File: keebach-narrow-v1.kicad_pcb (KiCad board)
At the start: 2 copper layers, 200 x 144.9 mm, 141 parts, among them J1 OLED_128x32, SW0 RotaryEncoder_Switch, SW1 RotaryEncoder_Switch, U0 RP2040-Matrix, U1 MCP23017x-x-SP, U2 TRRS, U3 TRRS

Commit message: Update PCB layout and schematic
Parts:
- added R0: 10k, Resistor_THT:R_Axial_DIN0207_L6.3mm_D2.5mm_P7.62mm_Horizontal, F.Cu at (134.6, 16.5)
- added R1: 10k, Resistor_THT:R_Axial_DIN0207_L6.3mm_D2.5mm_P7.62mm_Horizontal, F.Cu at (131.1, 16.5)
Connections:
- J1 pad 1: unconnected-(J1-GND-Pad1) -> GND
- J1 pad 2: unconnected-(J1-VCC-Pad2) -> 3V3
- J1 pad 3: unconnected-(J1-SCL-Pad3) -> SCL
- J1 pad 4: unconnected-(J1-SDA-Pad4) -> SDA
- U0 pad 1: 5V -> unconnected-(U0-5V-Pad1)
- U0 pad 13: unconnected-(U0-P3-Pad13) -> U0_TRRS
- U0 pad 14: unconnected-(U0-P4-Pad14) -> U1_TRRS
- U0 pad 8: U1_TRRS -> SCL
- U0 pad 9: U0_TRRS -> SDA
- U1 pad 10: unconnected-(U1-V_{SS}-Pad10) -> GND
- U1 pad 12: unconnected-(U1-SCK-Pad12) -> SCL
- U1 pad 13: unconnected-(U1-SDA-Pad13) -> SDA
- U1 pad 15: unconnected-(U1-A0-Pad15) -> GND
- U1 pad 16: unconnected-(U1-A1-Pad16) -> GND
- U1 pad 17: unconnected-(U1-A2-Pad17) -> GND
- U1 pad 18: unconnected-(U1-~{RESET}-Pad18) -> 3V3
- U1 pad 9: unconnected-(U1-V_{DD}-Pad9) -> 3V3
Routing:
- net 3V3: track 0.00 -> 89.9 mm, vias 0 -> 1
- net GND: track 290.8 -> 368.1 mm, vias 0 -> 2
- net SCL: track 0.00 -> 72.3 mm
- net SDA: track 0.00 -> 69.0 mm
- net U1_TRRS: track 87.1 -> 119.8 mm
- net COL_9: track 300.8 -> 309.3 mm
- net SW0_B: track 71.6 -> 77.7 mm
- net SW0_A: track 75.7 -> 81.2 mm
- net SW1_A: track 72.5 -> 77.0 mm
- net ROW_6: track 95.8 -> 100.1 mm
- net ROW_5: track 64.4 -> 68.7 mm
- net ROW_2: track 58.1 -> 62.3 mm
- net ROW_4: track 34.7 -> 38.8 mm
- net ROW_1: track 88.5 -> 92.6 mm
- net Net-(D61-A): track 220.5 -> 216.5 mm
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- added copper zone on B.Cu, net (none)
- added copper zone on F.Cu, net (none)
