File: keebach-narrow-v1.kicad_sch (KiCad schematic)
At the start: 141 parts, among them J1 OLED_128x32, SW0 RotaryEncoder_Switch, SW1 RotaryEncoder_Switch, U0 RP2040-Matrix, U1 MCP23017x-x-SP, U2 TRRS, U3 TRRS

Commit message: Wire MCP23017 power/address/reset/I2C bus and OLED hookup
Connects U1 (MCP23017) V_DD/V_SS/A0-A2/~RESET to 3V3/GND, routes
SCL/SDA to MCU pins P5/P3, ties the OLED (J1) into the same power
and I2C nets, and completes the R1/R2 pull-ups to 3V3. INTA/INTB
and the unused GPB3-7 expander pins are left spare intentionally.
Parts:
- added R1, R2: 10k, symbol Device:R
Connections:
- net 3V3: now also J1.2 (VCC), U1.18 (~{RESET}), U1.9 (V_{DD}), R1.2, R2.2
- net GND: now also J1.1 (GND), U1.10 (V_{SS}), U1.15 (A0), U1.16 (A1), U1.17 (A2)
- net SDA: now reaches U0.13 (P3)
- net SDA: now also J1.4 (SDA), U1.13 (SDA), R1.1
- net SCL: now reaches U0.15 (P5)
- net SCL: now also J1.3 (SCL), U1.12 (SCK), R2.1
- no-connect marks 5 -> 6

Commit message: Update PCB layout and schematic
Parts:
- R0: renamed from R1; footprint (none) -> Resistor_THT:R_Axial_DIN0207_L6.3mm_D2.5mm_P7.62mm_Horizontal
- R1: renamed from R2; footprint (none) -> Resistor_THT:R_Axial_DIN0207_L6.3mm_D2.5mm_P7.62mm_Horizontal
Connections:
- net SCL: now also U0.8 (P15); no longer U0.15 (P5)
- net SDA: now also U0.9 (P14); no longer U0.13 (P3)
- net U0_TRRS: now also U0.13 (P3); no longer U0.9 (P14)
- net U1_TRRS: now also U0.14 (P4); no longer U0.8 (P15)
- net 5V: no longer names the net of U0.1 (5V)
- no-connect marks 6 -> 9
Other:
- moved on the sheet: J1, R0, R1, U2, U3
